File: schematic/kicad/waxMelter.kicad_sch (KiCad schematic)
At the start: 17 parts, among them J1 Relay_Control_Terminal, SW1 PWR, SW2 T+, SW3 T-, U1 LD1117V33, U2 HUZZAH32_ESP32, U3 AD8495_Breakout, U4 AD8495_Breakout

Commit message: Add updated kicad files
Connections:
- net SENSOR_0: now also U2.19 (A2/GPI34); no longer U2.18 (A1/GPIO25)
- net SENSOR_1: now also U2.21 (A4/GPI36); no longer U2.22 (A5/GPIO4)
Other:
- note added: "NOTES: CIRCUIT REQUIRES 5V USB POWER SUPPLY CONNECTED TO HUZZAH32 AD8495_BREAKOUT TEMP(F) = (VOUT - 1.25)/0.009 + 32 SYSTEM CONTROLS EXTERNAL 120V LINE RELAY MODULE (ADAFRUIT 2935 ALL THERMOCOUPLES MUST BE K TYPE ESP32 SUPPORTS A2-A4, A9, A7 ONLY WITH WIFI ON"
- note removed: "NOTES: CIRCUIT REQUIRES 5V USB POWER SUPPLY CONNECTED TO HUZZAH32 AD8495_BREAKOUT TEMP(F) = (VOUT - 1.25)/0.009 + 32 SYSTEM CONTROLS EXTERNAL 120V LINE RELAY MODULE (ADAFRUIT 2935 ALL THERMOCOUPLES MUST BE K TYPE"
Changed lines of the file:
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@@
   (title_block
     (title "PID Thermocouple Controller for Wax Melting")
-    (date "2020-10-19")
-    (rev "Rev 1.0")
+    (date "2020-12-15")
+    (rev "Rev 1.1")
     (company "Maeve Stites & Co.")
   )
@@
   (junction (at 166.37 106.045) (diameter 1.016) (color 0 0 0 0))
   (junction (at 219.71 53.975) (diameter 1.016) (color 0 0 0 0))
+  (no_connect (at 73.66 123.19))
+  (no_connect (at 37.465 113.665))
+  (no_connect (at 37.465 147.955))
+  (no_connect (at 73.66 112.395))
+  (no_connect (at 48.26 102.87))
+  (no_connect (at 73.66 125.73))
+  (no_connect (at 37.465 140.335))
+  (no_connect (at 73.66 114.935))
+  (no_connect (at 37.465 125.73))
+  (no_connect (at 63.5 102.87))
   (no_connect (at 73.66 135.89))
+  (no_connect (at 37.465 142.875))
+  (no_connect (at 73.66 138.43))
+  (no_connect (at 37.465 120.65))
+  (no_connect (at 37.465 130.81))
+  (no_connect (at 37.465 145.415))
   (no_connect (at 37.465 137.795))
-  (no_connect (at 63.5 102.87))
-  (no_connect (at 37.465 113.665))
-  (no_connect (at 48.26 102.87))
   (no_connect (at 37.465 135.255))
-  (no_connect (at 37.465 140.335))
-  (no_connect (at 37.465 123.19))
-  (no_connect (at 73.66 112.395))
-  (no_connect (at 73.66 114.935))
-  (no_connect (at 73.66 125.73))
-  (no_connect (at 37.465 128.27))
-  (no_connect (at 37.465 145.415))
-  (no_connect (at 37.465 142.875))
-  (no_connect (at 37.465 125.73))
-  (no_connect (at 73.66 123.19))
-  (no_connect (at 73.66 138.43))
-  (no_connect (at 37.465 147.955))
   (wire (pts (xy 34.29 116.84) (xy 31.115 116.84))
     (stroke (width 0) (type solid) (color 0 0 0 0))
@@
     (stroke (width 0) (type solid) (color 0 0 0 0))
   )
-  (text "NOTES:\nCIRCUIT REQUIRES 5V USB POWER SUPPLY CONNECTED TO HUZZAH32\nAD8495_BREAKOUT TEMP(F) = (VOUT - 1.25)/0.009 + 32\nSYSTEM CONTROLS EXTERNAL 120V LINE RELAY MODULE (ADAFRUIT 2935\nALL THERMOCOUPLES MUST BE K TYPE"
-    (at 31.75 192.405 0)
+  (text "NOTES:\nCIRCUIT REQUIRES 5V USB POWER SUPPLY CONNECTED TO HUZZAH32\nAD8495_BREAKOUT TEMP(F) = (VOUT - 1.25)/0.009 + 32\nSYSTEM CONTROLS EXTERNAL 120V LINE RELAY MODULE (ADAFRUIT 2935\nALL THERMOCOUPLES MUST BE K TYPE\nESP32 SUPPORTS  A2-A4, A9, A7 ONLY WITH WIFI ON"
+    (at 31.369 195.453 0)
     (effects (font (size 2.032 2.032)) (justify left bottom))
   )
@@
     (effects (font (size 1.27 1.27)) (justify right))
   )
-  (global_label "SENSOR_0" (shape input) (at 37.465 120.65 180)
+  (global_label "SENSOR_0" (shape input) (at 37.465 123.19 180)
     (effects (font (size 1.27 1.27)) (justify right))
   )
-  (global_label "SENSOR_1" (shape input) (at 37.465 130.81 180)
+  (global_label "SENSOR_1" (shape input) (at 37.465 128.27 180)
     (effects (font (size 1.27 1.27)) (justify right))
   )
